Commit message: feat: add collision in urdf

File: src/kitty_bot_description/src/description/kitty_bot_description.urdf (robot description, URDF)
Before this commit: robot kitty_bot, 4 links, 3 joints
Links:
- link base_link: geometry collision cylinder length=${base_height} radius=${base_radius}; visual cylinder length=${base_height} radius=${base_radius}
- link behind_caster: geometry collision sphere radius=${caster_radius}; visual sphere radius=${caster_radius}
- link front_caster: geometry collision sphere radius=${caster_radius}; visual sphere radius=${caster_radius}

Commit message: feat: add lidar_link

File: src/kitty_bot_description/src/description/kitty_bot_description.urdf (robot description, URDF)
Before this commit: robot kitty_bot, 4 links, 3 joints
Links:
- added link lidar_link, mass 0.125; collision cylinder length=0.03 radius=0.03; visual cylinder length=0.03 radius=0.03
Joints:
- added joint lidar_joint: type fixed, parent base_link, child lidar_link, origin xyz=0 0 0.18 rpy=0 0 0
